Commit message: added stl of wheels

File: models/ackermann_model/ackermann_model.urdf (robot description, URDF)
Before this commit: robot ackermann_robot, 9 links, 8 joints
Links:
- link wheel_back_left: geometry collision cylinder length=0.04 radius=0.075; visual mesh filename=model://ackermann_model/meshes/wheel.stl scale=0.0055 0.0055 0.0055
- link wheel_back_right: geometry collision cylinder length=0.04 radius=0.075; visual mesh filename=model://ackermann_model/meshes/wheel.stl scale=0.0055 0.0055 0.0055
- link wheel_front_left: geometry collision cylinder length=0.04 radius=0.075; visual mesh filename=model://ackermann_model/meshes/wheel.stl scale=0.0055 0.0055 0.0055
- link wheel_front_right: geometry collision cylinder length=0.04 radius=0.075; visual mesh filename=model://ackermann_model/meshes/wheel.stl scale=0.0055 0.0055 0.0055
Joints:
- joint steering_wheel_front_left_joint: limit lower=-1e+16 upper=1e+16 effort=20.0 velocity=5.0 -> lower=-0.7 upper=0.7 effort=20.0 velocity=5.0
- joint steering_wheel_front_right_joint: limit lower=-1e+16 upper=1e+16 effort=20.0 velocity=5.0 -> lower=-0.7 upper=0.7 effort=20.0 velocity=5.0

File: urdf/ackermann_model.urdf.xacro (robot description, xacro)
@@ -42,15 +42,15 @@
   </gazebo>
 	<!-- The steering wheels -->
-	<xacro:steering_wheel name="front_left" parent="base_link" limit_low="-1e+16" limit_high="1e+16" >
+	<xacro:steering_wheel name="front_left" parent="base_link" limit_low="-0.7" limit_high="0.7" visual_roll="-${M_PI_2}" visual_y="-0.023" >
 		<origin xyz="0.308 0.175 -${wheel_radius}" rpy="0 0 0"/>
 	</xacro:steering_wheel>
-	<xacro:steering_wheel name="front_right" parent="base_link" limit_low="-1e+16" limit_high="1e+16" >
+	<xacro:steering_wheel name="front_right" parent="base_link" limit_low="-0.7" limit_high="0.7" visual_roll="${M_PI_2}" visual_y="0.025" >
 		<origin xyz="0.308 -0.175 -${wheel_radius}" rpy="0 0 0"/>
 	</xacro:steering_wheel>
 	<!-- wheels -->
-	<xacro:wheel name="back_left" parent="base_link" >
+	<xacro:wheel name="back_left" parent="base_link" visual_roll="-${M_PI_2}" visual_y="-0.023" >
 		<origin xyz="-0.308 0.175 -${wheel_radius}" rpy="0 0 0"/>
 	</xacro:wheel>
-	<xacro:wheel name="back_right" parent="base_link" >
+	<xacro:wheel name="back_right" parent="base_link" visual_roll="${M_PI_2}" visual_y="0.025" >
 		<origin xyz="-0.308 -0.175 -${wheel_radius}" rpy="0 0 0"/>
 	</xacro:wheel>
@@ -77,18 +77,14 @@
       <left_steering_joint>steering_wheel_front_left_joint</left_steering_joint>
       <right_steering_joint>steering_wheel_front_right_joint</right_steering_joint>
-      <!-- <steering_wheel_joint>steering_joint</steering_wheel_joint> -->
       <!-- Max absolute steer angle for tyre in radians-->
       <!-- Any cmd_vel angular z greater than this would be capped -->
-      <max_steer>0.6458</max_steer>
-      <!-- Max absolute steering angle of steering wheel -->
-      <!-- <max_steering_angle>7.85</max_steering_angle> -->
-      <!-- Max absolute linear speed in m/s -->
+      <max_steer>0.7</max_steer>
       <max_speed>20</max_speed>
       <!-- PID tuning -->
-      <left_steering_pid_gain>1500 0 1</left_steering_pid_gain>
+      <left_steering_pid_gain>75 0 1</left_steering_pid_gain>
       <left_steering_i_range>0 0</left_steering_i_range>
-      <right_steering_pid_gain>1500 0 1</right_steering_pid_gain>
+      <right_steering_pid_gain>75 0 1</right_steering_pid_gain>
       <right_steering_i_range>0 0</right_steering_i_range>
-      <linear_velocity_pid_gain>1000 0 1</linear_velocity_pid_gain>
+      <linear_velocity_pid_gain>50 0 1</linear_velocity_pid_gain>
       <linear_velocity_i_range>0 0</linear_velocity_i_range>
       <!-- output -->

File: urdf/steering_wheels.xacro (robot description, xacro)
@@ -2,5 +2,5 @@
 <robot name="steering_wheel" xmlns:xacro="http://ros.org/wiki/xacro">
   <!-- Steering -->
-  <xacro:macro name="steering_wheel" params="name parent *origin limit_low limit_high">
+  <xacro:macro name="steering_wheel" params="name parent *origin limit_low limit_high visual_roll visual_y">
     <link name="steering_wheel_${name}" >
 			<inertial>
@@ -22,5 +22,5 @@
       <dynamics damping="0.4" friction="0.5"/>
     </joint>
-		<xacro:wheel name="${name}" parent="steering_wheel_${name}">
+		<xacro:wheel name="${name}" parent="steering_wheel_${name}" visual_roll="${visual_roll}" visual_y="${visual_y}" >
 			<origin xyz="0.0 0.0 0.0" rpy="0 0 0"/>
 		</xacro:wheel>

File: urdf/wheels.xacro (robot description, xacro)
@@ -7,10 +7,10 @@
               izz="${m*r*r/2}"/>
   </xacro:macro>
-  <xacro:macro name="wheel" params="name parent *origin">
+  <xacro:macro name="wheel" params="name parent *origin visual_roll visual_y" >
     <link name="wheel_${name}">
       <visual>
-        <origin xyz="0 0 0" rpy="${M_PI_2} 0  0"/>
+        <origin xyz="0 ${visual_y} 0" rpy="${visual_roll} 0  0"/>
         <geometry>
-          <cylinder length="${wheel_height}" radius="${wheel_radius}"/>
+					<mesh filename="model://ackermann_model/meshes/wheel.stl" scale="0.0055 0.0055 0.0055" />
         </geometry>
         <material name="black"/>
